Commit message: add the .urdf file of washbasin

File: models/washbasin.urdf (robot description, URDF)
Before this commit: robot washbasin, 3 links, 2 joints
Links:
- link base_link: geometry collision box size=0.6 0.6 0.1; visual box size=0.6 0.6 0.1
- link basin_bowl: geometry collision cylinder length=0.3 radius=0.25; visual cylinder length=0.3 radius=0.25
Joints:
- joint base_to_basin: origin xyz=0 0 0.1 rpy=0 0 0 -> xyz=0 0 0.15 rpy=0 0 0
- joint basin_to_faucet: origin xyz=0 0 0.2 rpy=0 0 0 -> xyz=0 0 0.35 rpy=0 0 0
